File: PCB/Lathe RPM Display.sch (KiCad schematic (older format))
At the start: 18 parts, among them Q1 OH090U, Q2 2N7000, Q3 2N7000, Q4 2N7000, Q5 2N7000, U1 KCSC02-105, U2 KCSC02-105, U3 KCSC02-105, U4 KCSC02-105

Commit message: code, schematic and layout
Got code to a good working state. Schematic is good, maybe a couple more additions for power. Started layout and happy with locations. No traces routed.
Parts:
- added R9: 10k, Resistor_SMD:R_0805_2012Metric_Pad1.15x1.40mm_HandSolder, symbol Device:R_Small_US
- Q1: value OH090U -> A3144EU
- R1, R2, R3, R4, R5, R6, R7, R8: footprint (none) -> Resistor_SMD:R_0805_2012Metric_Pad1.15x1.40mm_HandSolder
- U1, U2, U3, U4: footprint Display_7Segment:KCSC02-105 -> Display_7Segment:7SegmentLED_LTS6760_LTS6780
Connections:
- wire segments 144 -> 153
- no-connect marks 0 -> 14
Changed lines of the file:
@@
 P 3250 1650
 F 0 "Q1" H 2922 1703 60  0000 R CNN
-F 1 "OH090U" H 2922 1597 60  0000 R CNN
+F 1 "A3144EU" H 2922 1597 60  0000 R CNN
 F 2 "digikey-footprints:TO-92-3" H 3450 1850 60  0001 L CNN
 F 3 "https://www.ttelectronics.com/TTElectronics/media/ProductFiles/Optoelectronics/Datasheets/OH090-OHS3100.pdf" H 3450 1950 60  0001 L CNN
@@
 F 0 "U1" H 6700 4217 50  0000 C CNN
 F 1 "KCSC02-105" H 6700 4126 50  0000 C CNN
-F 2 "Display_7Segment:KCSC02-105" H 6700 2950 50  0001 C CNN
+F 2 "Display_7Segment:7SegmentLED_LTS6760_LTS6780" H 6700 2950 50  0001 C CNN
 F 3 "http://www.kingbright.com/attachments/file/psearch/000/00/00/KCSC02-105(Ver.9A).pdf" H 6200 4025 50  0001 L CNN
 	1    6700 3550
@@
 	6400 3950 6000 3950
 Wire Wire Line
-	6000 3950 6000 2750
-Wire Wire Line
 	5800 2050 6350 2050
 Wire Wire Line
@@
 	6100 2550 6100 3750
 Wire Wire Line
-	5800 2650 6050 2650
-Wire Wire Line
 	6050 2650 6050 3850
-Wire Wire Line
-	5800 2750 6000 2750
 $Comp
 L Display_Character:KCSC02-105 U2
@@
 F 0 "U2" H 7800 4217 50  0000 C CNN
 F 1 "KCSC02-105" H 7800 4126 50  0000 C CNN
-F 2 "Display_7Segment:KCSC02-105" H 7800 2950 50  0001 C CNN
+F 2 "Display_7Segment:7SegmentLED_LTS6760_LTS6780" H 7800 2950 50  0001 C CNN
 F 3 "http://www.kingbright.com/attachments/file/psearch/000/00/00/KCSC02-105(Ver.9A).pdf" H 7300 4025 50  0001 L CNN
 	1    7800 3550
@@
 Wire Wire Line
 	7150 3850 7500 3850
-Connection ~ 6050 2650
-Wire Wire Line
-	6000 2750 7100 2750
 Wire Wire Line
 	7100 2750 7100 3950
 Wire Wire Line
 	7100 3950 7500 3950
-Connection ~ 6000 2750
 $Comp
 L Device:R_Small_US R1
@@
 F 0 "R1" V 5650 1950 40  0000 C CNN
 F 1 "470" V 5650 2150 40  0000 C CNN
-F 2 "" H 5700 2050 50  0001 C CNN
+F 2 "Resistor_SMD:R_0805_2012Metric_Pad1.15x1.40mm_HandSolder" H 5700 2050 50  0001 C CNN
 F 3 "~" H 5700 2050 50  0001 C CNN
 	1    5700 2050
@@
 Wire Wire Line
 	5600 2550 5350 2550
-Wire Wire Line
-	5600 2650 5350 2650
-Wire Wire Line
-	5600 2750 5350 2750
 $Comp
 L Device:R_Small_US R2
@@
 F 0 "R2" V 5650 2050 40  0000 C CNN
 F 1 "470" V 5650 2250 40  0000 C CNN
-F 2 "" H 5700 2150 50  0001 C CNN
+F 2 "Resistor_SMD:R_0805_2012Metric_Pad1.15x1.40mm_HandSolder" H 5700 2150 50  0001 C CNN
 F 3 "~" H 5700 2150 50  0001 C CNN
 	1    5700 2150
@@
 F 0 "R3" V 5650 2150 40  0000 C CNN
 F 1 "470" V 5650 2350 40  0000 C CNN
-F 2 "" H 5700 2250 50  0001 C CNN
+F 2 "Resistor_SMD:R_0805_2012Metric_Pad1.15x1.40mm_HandSolder" H 5700 2250 50  0001 C CNN
 F 3 "~" H 5700 2250 50  0001 C CNN
 	1    5700 2250
@@
 F 0 "R4" V 5650 2250 40  0000 C CNN
 F 1 "470" V 5650 2450 40  0000 C CNN
-F 2 "" H 5700 2350 50  0001 C CNN
+F 2 "Resistor_SMD:R_0805_2012Metric_Pad1.15x1.40mm_HandSolder" H 5700 2350 50  0001 C CNN
 F 3 "~" H 5700 2350 50  0001 C CNN
 	1    5700 2350
@@
 F 0 "R5" V 5650 2350 40  0000 C CNN
 F 1 "470" V 5650 2550 40  0000 C CNN
-F 2 "" H 5700 2450 50  0001 C CNN
+F 2 "Resistor_SMD:R_0805_2012Metric_Pad1.15x1.40mm_HandSolder" H 5700 2450 50  0001 C CNN
 F 3 "~" H 5700 2450 50  0001 C CNN
 	1    5700 2450
@@
 F 0 "R6" V 5650 2450 40  0000 C CNN
 F 1 "470" V 5650 2650 40  0000 C CNN
-F 2 "" H 5700 2550 50  0001 C CNN
+F 2 "Resistor_SMD:R_0805_2012Metric_Pad1.15x1.40mm_HandSolder" H 5700 2550 50  0001 C CNN
 F 3 "~" H 5700 2550 50  0001 C CNN
 	1    5700 2550
@@
 L Device:R_Small_US R7
 U 1 1 5DD19451
-P 5700 2650
-F 0 "R7" V 5650 2550 40  0000 C CNN
-F 1 "470" V 5650 2750 40  0000 C CNN
-F 2 "" H 5700 2650 50  0001 C CNN
-F 3 "~" H 5700 2650 50  0001 C CNN
-	1    5700 2650
+P 5650 3850
+F 0 "R7" V 5600 3750 40  0000 C CNN
+F 1 "470" V 5600 3950 40  0000 C CNN
+F 2 "Resistor_SMD:R_0805_2012Metric_Pad1.15x1.40mm_HandSolder" H 5650 3850 50  0001 C CNN
+F 3 "~" H 5650 3850 50  0001 C CNN
+	1    5650 3850
 	0    1    1    0
 $EndComp
@@
 L Device:R_Small_US R8
 U 1 1 5DD19477
-P 5700 2750
-F 0 "R8" V 5650 2650 40  0000 C CNN
-F 1 "470" V 5650 2850 40  0000 C CNN
-F 2 "" H 5700 2750 50  0001 C CNN
-F 3 "~" H 5700 2750 50  0001 C CNN
-	1    5700 2750
+P 5650 3950
+F 0 "R8" V 5600 3850 40  0000 C CNN
+F 1 "470" V 5600 4050 40  0000 C CNN
+F 2 "Resistor_SMD:R_0805_2012Metric_Pad1.15x1.40mm_HandSolder" H 5650 3950 50  0001 C CNN
+F 3 "~" H 5650 3950 50  0001 C CNN
+	1    5650 3950
 	0    1    1    0
 $EndComp
@@
 F 0 "U3" H 8900 4217 50  0000 C CNN
 F 1 "KCSC02-105" H 8900 4126 50  0000 C CNN
-F 2 "Display_7Segment:KCSC02-105" H 8900 2950 50  0001 C CNN
+F 2 "Display_7Segment:7SegmentLED_LTS6760_LTS6780" H 8900 2950 50  0001 C CNN
 F 3 "http://www.kingbright.com/attachments/file/psearch/000/00/00/KCSC02-105(Ver.9A).pdf" H 8400 4025 50  0001 L CNN
 	1    8900 3550
@@
 Wire Wire Line
 	8200 3950 8600 3950
-Connection ~ 7100 2750
 $Comp
 L Display_Character:KCSC02-105 U4
@@
 F 0 "U4" H 10000 4217 50  0000 C CNN
 F 1 "KCSC02-105" H 10000 4126 50  0000 C CNN
-F 2 "Display_7Segment:KCSC02-105" H 10000 2950 50  0001 C CNN
+F 2 "Display_7Segment:7SegmentLED_LTS6760_LTS6780" H 10000 2950 50  0001 C CNN
 F 3 "http://www.kingbright.com/attachments/file/psearch/000/00/00/KCSC02-105(Ver.9A).pdf" H 9500 4025 50  0001 L CNN
 	1    10000 3550
@@
 Text Label 5400 2550 0    50   ~ 0
 F
-Text Label 5400 2650 0    50   ~ 0
+Text Label 4300 2850 1    50   ~ 0
 G
-Text Label 5400 2750 0    50   ~ 0
+Text Label 4200 2850 1    50   ~ 0
 DP
 Wire Wire Line
-	4350 1650 3650 1650
+	4350 1650 3700 1650
 $Comp
 L Transistor_FET:2N7000 Q2
@@
 	10350 6000 10350 5950
 Wire Wire Line
-	6750 4250 4200 4250
-Wire Wire Line
-	4200 4250 4200 2150
-Wire Wire Line
-	4200 2150 4350 2150
-Wire Wire Line
-	4350 2050 4100 2050
-Wire Wire Line
-	4100 2050 4100 4750
-Wire Wire Line
-	4100 4750 7850 4750
-Wire Wire Line
-	4350 1950 4000 1950
-Wire Wire Line
-	4000 1950 4000 5250
-Wire Wire Line
-	4000 5250 8950 5250
-Wire Wire Line
-	10050 5750 3900 5750
-Wire Wire Line
-	3900 5750 3900 1850
-Wire Wire Line
-	3900 1850 4350 1850
-$Comp
-L power:GND #PWR?
+	6750 4250 4100 4250
+Wire Wire Line
+	4100 4250 4100 2150
+Wire Wire Line
+	4100 2150 4350 2150
+Wire Wire Line
+	4350 2050 4000 2050
+Wire Wire Line
+	4000 2050 4000 4750
+Wire Wire Line
+	4000 4750 7850 4750
+Wire Wire Line
+	4350 1950 3900 1950
+Wire Wire Line
+	3900 1950 3900 5250
+Wire Wire Line
+	3900 5250 8950 5250
+Wire Wire Line
+	10050 5750 3800 5750
+Wire Wire Line
+	3800 5750 3800 1850
+Wire Wire Line
+	3800 1850 4350 1850
+$Comp
+L power:GND #PWR04
 U 1 1 5DD242B8
 P 4850 3150
-F 0 "#PWR?" H 4850 2900 50  0001 C CNN
+F 0 "#PWR04" H 4850 2900 50  0001 C CNN
 F 1 "GND" H 4855 2977 50  0000 C CNN
 F 2 "" H 4850 3150 50  0001 C CNN
@@
 $EndComp
 $Comp
-L power:GND #PWR?
+L power:GND #PWR01
 U 1 1 5DD242E7
 P 3050 1950
-F 0 "#PWR?" H 3050 1700 50  0001 C CNN
+F 0 "#PWR01" H 3050 1700 50  0001 C CNN
 F 1 "GND" H 3055 1777 50  0000 C CNN
 F 2 "" H 3050 1950 50  0001 C CNN
@@
 $EndComp
 $Comp
-L power:+5V #PWR?
+L power:+5V #PWR02
 U 1 1 5DD2439D
 P 3150 1350
-F 0 "#PWR?" H 3150 1200 50  0001 C CNN
+F 0 "#PWR02" H 3150 1200 50  0001 C CNN
 F 1 "+5V" H 3165 1523 50  0000 C CNN
 F 2 "" H 3150 1350 50  0001 C CNN
@@
 $EndComp
 $Comp
-L power:+5V #PWR?
+L power:+5V #PWR03
 U 1 1 5DD243D3
 P 4750 950
-F 0 "#PWR?" H 4750 800 50  0001 C CNN
+F 0 "#PWR03" H 4750 800 50  0001 C CNN
 F 1 "+5V" H 4765 1123 50  0000 C CNN
 F 2 "" H 4750 950 50  0001 C CNN
@@
 $EndComp
 Wire Wire Line
-	3150 1450 3150 1350
+	3150 1450 3150 1400
 Wire Wire Line
 	3050 1950 3050 1850
@@
 Wire Wire Line
 	4750 950  4750 1050
+Wire Wire Line
+	3700 1650 3700 1400
+Connection ~ 3700 1650
+Wire Wire Line
+	3700 1650 3650 1650
+$Comp
+L Device:R_Small_US R9
+U 1 1 5DDAFEF5
+P 3450 1400
+F 0 "R9" V 3400 1300 40  0000 C CNN
+F 1 "10k" V 3400 1500 40  0000 C CNN
+F 2 "Resistor_SMD:R_0805_2012Metric_Pad1.15x1.40mm_HandSolder" H 3450 1400 50  0001 C CNN
+F 3 "~" H 3450 1400 50  0001 C CNN
+	1    3450 1400
+	0    1    1    0
+$EndComp
+Wire Wire Line
+	3700 1400 3550 1400
+Wire Wire Line
+	3350 1400 3150 1400
+Connection ~ 3150 1400
+Wire Wire Line
+	3150 1400 3150 1350
+Connection ~ 7100 2750
+Wire Wire Line
+	6000 2750 7100 2750
+Wire Wire Line
+	5750 3950 6000 3950
+Connection ~ 6000 3950
+Wire Wire Line
+	6000 3950 6000 2750
+Wire Wire Line
+	5750 3850 6050 3850
+Connection ~ 6050 3850
+Wire Wire Line
+	5550 3850 4300 3850
+Wire Wire Line
+	4300 3850 4300 2750
+Wire Wire Line
+	4300 2750 4350 2750
+Wire Wire Line
+	4200 3950 4200 2650
+Wire Wire Line
+	4200 2650 4350 2650
+Wire Wire Line
+	4200 3950 5550 3950
+NoConn ~ 4350 1450
+NoConn ~ 4350 1550
+NoConn ~ 4350 1750
+NoConn ~ 4350 2250
+NoConn ~ 4350 2350
+NoConn ~ 4350 2450
+NoConn ~ 4350 2550
+NoConn ~ 5350 2750
+NoConn ~ 5350 2650
+NoConn ~ 5350 1850
+NoConn ~ 5350 1550
+NoConn ~ 5350 1450
+NoConn ~ 4950 1050
+NoConn ~ 5050 1050
 $EndSCHEMATC

Commit message: hall effect fix
Adjusted pulses per revolution to fix hall effect sensor double pulse
Parts:
- added J1: Conn_01x02, Connector_PinSocket_2.54mm:PinSocket_1x02_P2.54mm_Vertical, symbol Connector_Generic:Conn_01x02
Connections:
- wire segments 153 -> 157
Changed lines of the file:
@@
 encoding utf-8
 Sheet 1 1
-Title ""
-Date ""
-Rev ""
+Title "Lathe RPM Display"
+Date "2020-01-05"
+Rev "A"
 Comp ""
 Comment1 ""
@@
 	10350 6000 10350 5950
 Wire Wire Line
-	6750 4250 4100 4250
-Wire Wire Line
-	4100 4250 4100 2150
+	8950 5250 4100 5250
+Wire Wire Line
+	4100 5250 4100 2150
 Wire Wire Line
 	4100 2150 4350 2150
@@
 	4350 2050 4000 2050
 Wire Wire Line
-	4000 2050 4000 4750
-Wire Wire Line
-	4000 4750 7850 4750
+	4000 2050 4000 5750
+Wire Wire Line
+	4000 5750 10050 5750
 Wire Wire Line
 	4350 1950 3900 1950
 Wire Wire Line
-	3900 1950 3900 5250
-Wire Wire Line
-	3900 5250 8950 5250
-Wire Wire Line
-	10050 5750 3800 5750
-Wire Wire Line
-	3800 5750 3800 1850
+	3900 1950 3900 4250
+Wire Wire Line
+	7850 4750 3800 4750
+Wire Wire Line
+	3800 4750 3800 1850
 Wire Wire Line
 	3800 1850 4350 1850
@@
 	5750 3850 6050 3850
 Connection ~ 6050 3850
-Wire Wire Line
-	5550 3850 4300 3850
-Wire Wire Line
-	4300 3850 4300 2750
-Wire Wire Line
-	4300 2750 4350 2750
 Wire Wire Line
 	4200 3950 4200 2650
@@
 NoConn ~ 4950 1050
 NoConn ~ 5050 1050
+Wire Wire Line
+	3900 4250 6750 4250
+$Comp
+L Connector_Generic:Conn_01x02 J1
+U 1 1 5E11F0AC
+P 3300 3100
+F 0 "J1" H 3300 2900 50  0000 C CNN
+F 1 "Conn_01x02" H 2750 3050 50  0000 C CNN
+F 2 "Connector_PinSocket_2.54mm:PinSocket_1x02_P2.54mm_Vertical" H 3300 3100 50  0001 C CNN
+F 3 "~" H 3300 3100 50  0001 C CNN
+	1    3300 3100
+	1    0    0    1
+$EndComp
+$Comp
+L power:+5V #PWR0105
+U 1 1 5E11F252
+P 3050 2950
+F 0 "#PWR0105" H 3050 2800 50  0001 C CNN
+F 1 "+5V" H 3065 3123 50  0000 C CNN
+F 2 "" H 3050 2950 50  0001 C CNN
+F 3 "" H 3050 2950 50  0001 C CNN
+	1    3050 2950
+	1    0    0    -1
+$EndComp
+$Comp
+L power:GND #PWR0106
+U 1 1 5E11F285
+P 3050 3150
+F 0 "#PWR0106" H 3050 2900 50  0001 C CNN
+F 1 "GND" H 3055 2977 50  0000 C CNN
+F 2 "" H 3050 3150 50  0001 C CNN
+F 3 "" H 3050 3150 50  0001 C CNN
+	1    3050 3150
+	1    0    0    -1
+$EndComp
+Wire Wire Line
+	3100 3000 3050 3000
+Wire Wire Line
+	3050 3000 3050 2950
+Wire Wire Line
+	3100 3100 3050 3100
+Wire Wire Line
+	3050 3100 3050 3150
+Wire Wire Line
+	5550 3850 4300 3850
+Wire Wire Line
+	4300 2750 4350 2750
+Wire Wire Line
+	4300 2750 4300 3850
 $EndSCHEMATC
